File: nametag_smd.sch (KiCad schematic (older format))
At the start: 116 parts, among them IC1 ATTINY13-S, P1 ISP, Q1 2N7002, Q2 2N7002, Q3 2N7002, Q4 2N7002, Q5 2N7002

Commit message: Changed the package variant of the ATTINY13 to SO-8 narrow (ATTINY13-SS) because it is cheaper.
Fixed wrong ISP pinning.

Cleaned up the older thiner pcb tracks.
Parts:
- removed IC1: ATTINY13-S, nametag:SOIC-8-N_HandSoldering, symbol ATTINY13-S
- added IC1: ATTINY13-SS, SMD_Packages:SOIC-8-N, symbol ATTINY13-SS
Connections:
- wire segments 39 -> 40
- no-connect marks 1 -> 0
Other:
- moved on the sheet: P1
Changed lines of the file:
@@
 P 2200 2100
 F 0 "Q1" H 2500 2150 50  0000 R CNN
-F 1 "2N7002" H 2850 2050 50  0000 R CNN
+F 1 "2N7002" H 2700 2000 50  0000 R CNN
 F 2 "TO_SOT_Packages_SMD:SOT-23_Handsoldering" H 2400 2200 50  0001 C CNN
 F 3 "" H 2200 2100 50  0000 C CNN
@@
 L CONN_02X03 P1
 U 1 1 570B1B1B
-P 2100 6650
-F 0 "P1" H 2100 6850 50  0000 C CNN
-F 1 "ISP" H 2100 6450 50  0000 C CNN
-F 2 "Pin_Headers:Pin_Header_Straight_2x03" H 2100 5450 50  0001 C CNN
-F 3 "" H 2100 5450 50  0000 C CNN
-	1    2100 6650
+P 2100 6750
+F 0 "P1" H 2100 6950 50  0000 C CNN
+F 1 "ISP" H 2100 6550 50  0000 C CNN
+F 2 "Pin_Headers:Pin_Header_Straight_2x03" H 2100 5550 50  0001 C CNN
+F 3 "" H 2100 5550 50  0000 C CNN
+	1    2100 6750
 	-1   0    0    -1
 $EndComp
-Text Label 1750 6550 2    60   ~ 0
+Text Label 1750 6650 2    60   ~ 0
 MOSI
-Text Label 2350 6550 0    60   ~ 0
+Text Label 2350 6650 0    60   ~ 0
 MISO
-Text Label 2350 6650 0    60   ~ 0
+Text Label 2350 6750 0    60   ~ 0
 SCK
-Text Label 2350 6750 0    60   ~ 0
+Text Label 2350 6850 0    60   ~ 0
 ~RESET
 Text Label 3400 5900 2    60   ~ 0
@@
 L GND #PWR06
 U 1 1 570B36D8
-P 1850 6850
-F 0 "#PWR06" H 1850 6600 50  0001 C CNN
-F 1 "GND" H 1850 6700 50  0000 C CNN
-F 2 "" H 1850 6850 50  0000 C CNN
-F 3 "" H 1850 6850 50  0000 C CNN
-	1    1850 6850
+P 1850 6950
+F 0 "#PWR06" H 1850 6700 50  0001 C CNN
+F 1 "GND" H 1850 6800 50  0000 C CNN
+F 2 "" H 1850 6950 50  0000 C CNN
+F 3 "" H 1850 6950 50  0000 C CNN
+	1    1850 6950
 	-1   0    0    -1
 $EndComp
@@
 P 2200 2700
 F 0 "Q2" H 2500 2750 50  0000 R CNN
-F 1 "2N7002" H 2850 2650 50  0000 R CNN
+F 1 "2N7002" H 2700 2600 50  0000 R CNN
 F 2 "TO_SOT_Packages_SMD:SOT-23_Handsoldering" H 2400 2800 50  0001 C CNN
 F 3 "" H 2200 2700 50  0000 C CNN
@@
 P 2200 3300
 F 0 "Q3" H 2500 3350 50  0000 R CNN
-F 1 "2N7002" H 2850 3250 50  0000 R CNN
+F 1 "2N7002" H 2700 3200 50  0000 R CNN
 F 2 "TO_SOT_Packages_SMD:SOT-23_Handsoldering" H 2400 3400 50  0001 C CNN
 F 3 "" H 2200 3300 50  0000 C CNN
@@
 P 2200 3900
 F 0 "Q4" H 2500 3950 50  0000 R CNN
-F 1 "2N7002" H 2850 3850 50  0000 R CNN
+F 1 "2N7002" H 2700 3800 50  0000 R CNN
 F 2 "TO_SOT_Packages_SMD:SOT-23_Handsoldering" H 2400 4000 50  0001 C CNN
 F 3 "" H 2200 3900 50  0000 C CNN
@@
 P 2200 4500
 F 0 "Q5" H 2500 4550 50  0000 R CNN
-F 1 "2N7002" H 2850 4450 50  0000 R CNN
+F 1 "2N7002" H 2700 4400 50  0000 R CNN
 F 2 "TO_SOT_Packages_SMD:SOT-23_Handsoldering" H 2400 4600 50  0001 C CNN
 F 3 "" H 2200 4500 50  0000 C CNN
@@
 	3700 4900 3700 5000
 Wire Wire Line
-	1850 6850 1850 6750
+	1850 6950 1850 6850
 Wire Wire Line
 	6300 5800 6300 6000
@@
 	4200 6300 1750 6300
 Wire Wire Line
-	1750 6300 1750 6550
-Wire Wire Line
-	1750 6550 1850 6550
-Wire Wire Line
-	4100 6550 2350 6550
-Wire Wire Line
-	4000 6650 2350 6650
+	1750 6300 1750 6750
+Wire Wire Line
+	4100 6650 2350 6650
+Wire Wire Line
+	4000 6750 2350 6750
 Connection ~ 3900 5900
 Wire Wire Line
 	4200 5400 4200 6300
 Wire Wire Line
-	4100 5500 4100 6550
-Wire Wire Line
-	4000 5600 4000 6650
+	4100 5500 4100 6650
+Wire Wire Line
+	4000 5600 4000 6750
 $Comp
 L GND #PWR017
@@
 $EndComp
 Wire Wire Line
-	3900 5900 3900 6750
-Wire Wire Line
-	3900 6750 2350 6750
+	3900 5900 3900 6850
+Wire Wire Line
+	3900 6850 2350 6850
 Wire Wire Line
 	2350 6000 2350 5900
@@
 Text Notes 7450 5700 0    60   ~ 0
 Coincell battery holder\nCR2032
-NoConn ~ 1850 6650
 Wire Wire Line
 	6300 5300 6300 5500
 Connection ~ 6300 5400
 $Comp
-L ATTINY13-S IC1
-U 1 1 574F459B
+L ATTINY13-SS IC1
+U 1 1 57553A6D
 P 5300 5650
 F 0 "IC1" H 4500 6050 50  0000 C CNN
-F 1 "ATTINY13-S" H 5950 5250 50  0000 C CNN
-F 2 "nametag:SOIC-8-N_HandSoldering" H 5950 5650 50  0001 C CIN
+F 1 "ATTINY13-SS" H 5950 5250 50  0000 C CNN
+F 2 "SMD_Packages:SOIC-8-N" H 5900 5650 50  0001 C CIN
 F 3 "" H 4500 6000 50  0000 C CNN
 	1    5300 5650
 	1    0    0    -1
 $EndComp
+Wire Wire Line
+	1750 6750 1850 6750
+$Comp
+L VCC #PWR?
+U 1 1 5757BCC2
+P 1850 6550
+F 0 "#PWR?" H 1850 6400 50  0001 C CNN
+F 1 "VCC" H 1850 6700 50  0000 C CNN
+F 2 "" H 1850 6550 50  0000 C CNN
+F 3 "" H 1850 6550 50  0000 C CNN
+	1    1850 6550
+	1    0    0    -1
+$EndComp
+Wire Wire Line
+	1850 6650 1850 6550
 $EndSCHEMATC
